File: PCB/Main Boards/OSO-SWAT-B1/OSO-SWAT-B1.kicad_pcb (KiCad board)
At the start: 2 copper layers, 24.4 x 24.4 mm, 37 parts, among them J1 OSO_SWD, U1 ATSAML22J18A-MUT, U2 MIC5365-3.3YC5-TR, X1 Crystal

Commit message: WIP buzzer protection
Parts:
- R1: value DNP -> TBD
Connections:
- R1 pad 1: VCC -> /BUZZER
- R1 pad 2: /~{RESET} -> /BUZZER_SAFE
- U1 pad 51: /BUZZER -> /BUZZER_SAFE
Routing:
- net /BUZZER: track 7.69 -> 5.18 mm
- net /BUZZER_SAFE: track 0.00 -> 2.03 mm
- net /~{RESET}: track 24.6 -> 23.7 mm
Other:
- board text added: "SWAT-B1-02"
- board text removed: "SWAT-B1-01"
