File: PCB/Main Boards/OSO-SWAT-B1/OSO-SWAT-B1-jig/OSO-SWAT-B1-jig.kicad_pcb (KiCad board)
At the start: 2 copper layers, 44.5 x 46.9 mm, 31 parts, among them J1 TP7/A1_SCK, J10 TP1/VLCD, J11 TP11/~{RESET}, J12 GND, J13 GND, J2 TP6/A4{slash}D1{slash}MISO, J3 TP10/ALARM, J4 TP3/GND, J5 TP8/LIGHT, J6 TP9/MODE, J7 TP5/SWCLK, J8 TP2/SWDIO, J9 TP4/VCC

Commit message: SWL jig
Parts:
- J1: value TP7/A1_SCK -> TP1/VLCD
- J10: value TP1/VLCD -> TP10/ALARM
- J13: value GND -> Conn_01x27_Pin; footprint Connector_PinHeader_2.54mm:PinHeader_1x01_P2.54mm_Vertical -> OSO-SWAT-C1:testjig-zebra-footprint
- J2: value TP6/A4/D1/MISO -> TP2/SWDIO
- J3: value TP10/ALARM -> TP3/GND
- J4: value TP3/GND -> TP4/VCC
- J5: value TP8/LIGHT -> TP5/SWCLK
- J6: value TP9/MODE -> TP6/A4/D1/MISO
- J7: value TP5/SWCLK -> TP7/A1_SCK
- J8: value TP2/SWDIO -> TP8/LIGHT
- J9: value TP4/VCC -> TP9/MODE
- moved J13 33.9 mm to (62.1, 72.5)
- moved J10 16.5 mm to (71.2, 42.3)
- moved J6 11.4 mm to (61.0, 42.3)
- moved J11 8.89 mm to (73.7, 42.3)
- moved J8 8.89 mm to (66.1, 42.3)
- moved J3 6.35 mm to (53.4, 42.3)
- moved J4 6.35 mm to (55.9, 42.3)
- moved J7 3.81 mm to (63.5, 42.3)
- moved J9 1.27 mm to (68.6, 42.3)
- moved J5 1.27 mm to (58.5, 42.3)
- moved J1 1.27 mm to (48.3, 42.3)
- moved J12 1.27 mm to (76.2, 42.3)
- moved J2 1.27 mm to (50.8, 42.3)
Connections:
- J1 pad 1: A1_SCK -> VLCD
- J10 pad 1: VLCD -> ALARM
- J13 pad 1: GND -> unconnected-(J13-Pin_1-Pad1)
- J2 pad 1: A4/D1/MISO -> SWDIO
- J3 pad 1: ALARM -> GND
- J4 pad 1: GND -> VCC
- J5 pad 1: LIGHT -> SWCLK
- J6 pad 1: MODE -> A4/D1/MISO
- J7 pad 1: SWCLK -> A1_SCK
- J8 pad 1: SWDIO -> LIGHT
- J9 pad 1: VCC -> MODE
- N1 pad 1: (no net) -> unconnected-(N1-Pad1)
- N2 pad 1: (no net) -> unconnected-(N2-Pad1)
- N3 pad 1: (no net) -> unconnected-(N3-Pad1)
- N4 pad 1: (no net) -> unconnected-(N4-Pad1)
Routing:
- net GND: track 52.4 -> 0.00 mm
- net A1_SCK: track 44.9 -> 0.00 mm
- net A4/D1/MISO: track 44.9 -> 0.00 mm
- net MODE: track 41.6 -> 0.00 mm
- net SWDIO: track 40.8 -> 0.00 mm
- net ALARM: track 40.7 -> 0.00 mm
- net VCC: track 38.8 -> 0.00 mm
- net SWCLK: track 36.3 -> 0.00 mm
- net ~{RESET}: track 33.6 -> 0.00 mm
- net LIGHT: track 22.4 -> 0.00 mm
- net VLCD: track 20.5 -> 0.00 mm
